Commit message: Add parameters and update visual

File: marvin_simulation/urdf/depth_camera.xacro (robot description, xacro)
@@ -1,41 +1,36 @@
 <?xml version="1.0"?>
 <robot xmlns:xacro="http://ros.org/wiki/xacro" name="depth_camera">
-    <xacro:macro name="camera" params="mass *joint_origin">
-        <link name="camera">
-            <inertial>
-                <mass value="${camera_mass}"/>
-                <origin xyz="0 0 0" rpy="0 0 0"/>
-                <inertia
-                    ixx="1e-6" ixy="0.0" ixz="0.0"
-                    iyy="1e-6" iyz="0.0"
-                    izz="1e-6"
-                  />
-            </inertial>
+    <xacro:macro name="depth_camera" params="prefix mass length width height parent *joint_origin">
+        <xacro:include filename="$(find marvin_simulation)/urdf/inertia.xacro"/>
+        <link name="${prefix}_depth_camera">
+            <xacro:box_inertia mass="${mass}" length="${length}" width="${width}" height="${height}">
+                <origin xyz="0 0 ${height/2}" rpy="0 0 0" />
+            </xacro:box_inertia>
             <visual>
-                <origin xyz="0 0 0" rpy="0 0 0"/>
+                <origin xyz="0 0 ${height/2}" rpy="0 0 0"/>
                 <geometry>
-                    <box size="0.05 0.05 0.03"/>
+                    <box size="${length} ${width} ${height}"/>
                 </geometry>
             </visual>
             <collision>
-                <origin xyz="0 0 0" rpy="0 0 0"/>
+                <origin xyz="0 0 ${height/2}" rpy="0 0 0"/>
                 <geometry>
-                    <box size="0.05 0.05 0.03"/>
+                    <box size="${length} ${width} ${height}"/>
                 </geometry>
             </collision>
         </link>
-        <link name="camera_link_optical" />
-        <joint name="sim_camera_joint" type="fixed">
+        <link name="${prefix}_depth_camera_optical_link" />
+        <joint name="${prefix}_depth_camera_optical_joint" type="fixed">
+            <origin xyz="0 0 0" rpy="${-pi/2} 0 ${-pi/2}"/>
+            <parent link="${prefix}_depth_camera" />
+            <child link="${prefix}_depth_camera_optical_link" />
+        </joint>
+        <joint name="${prefix}_depth_camera_joint" type="fixed">
             <xacro:insert_block name="joint_origin" />
-            <parent link="base_link" />
-            <child link="camera" />
+            <parent link="${parent}" />
+            <child link="${prefix}_depth_camera" />
             <axis xyz="0 1 0" />
         </joint>
-        <joint name="camera_optical_joint" type="fixed">
-            <origin xyz="0 0 0" rpy="${-pi/2} 0 ${-pi/2}"/>
-            <parent link="camera" />
-            <child link="camera_link_optical" />
-        </joint>
-        <gazebo reference="camera">
+        <gazebo reference="${prefix}_depth_camera">
             <material>Gazebo/Yellow</material>
         </gazebo>

File: marvin_simulation/urdf/marvin.xacro (robot description, xacro)
@@ -134,7 +134,7 @@
     <!-- Sim Camera -->
 	<xacro:include filename="$(find marvin_simulation)/urdf/depth_camera.xacro" />
-	<xacro:camera mass="${camera_mass}">
+	<xacro:depth_camera prefix="zed" mass="${camera_mass}" length = "${1.5*0.0254}" width="${6.75*0.0254}" height="${1*0.0254}" parent="base_link">
 		<origin xyz="${camera_x_offset} 0 ${camera_z_offset}" rpy="0 ${camera_angle} 0" />
-	</xacro:camera>
+	</xacro:depth_camera>
     <!-- Lidar -->
     <xacro:include filename="$(find velodyne_description)/urdf/VLP-16.urdf.xacro" />

Commit message: Add depth_camera_base_link to implement proper cam view and mounting

File: marvin_simulation/urdf/depth_camera.xacro (robot description, xacro)
@@ -1,12 +1,12 @@
 <?xml version="1.0"?>
 <robot xmlns:xacro="http://ros.org/wiki/xacro" name="depth_camera">
-    <xacro:macro name="depth_camera" params="prefix mass length width height parent *joint_origin">
+    <xacro:macro name="depth_camera" params="prefix mass length width height parent:=base_link *joint_origin">
         <xacro:include filename="$(find marvin_simulation)/urdf/inertia.xacro"/>
-        <link name="${prefix}_depth_camera">
+        <link name="${prefix}_depth_camera_link">
             <xacro:box_inertia mass="${mass}" length="${length}" width="${width}" height="${height}">
-                <origin xyz="0 0 ${height/2}" rpy="0 0 0" />
+                <origin xyz="0 0 0" rpy="0 0 0" />
             </xacro:box_inertia>
             <visual>
-                <origin xyz="0 0 ${height/2}" rpy="0 0 0"/>
+                <origin xyz="0 0 0" rpy="0 0 0"/>
                 <geometry>
                     <box size="${length} ${width} ${height}"/>
@@ -14,5 +14,5 @@
             </visual>
             <collision>
-                <origin xyz="0 0 ${height/2}" rpy="0 0 0"/>
+                <origin xyz="0 0 0" rpy="0 0 0"/>
                 <geometry>
                     <box size="${length} ${width} ${height}"/>
@@ -23,11 +23,17 @@
         <joint name="${prefix}_depth_camera_optical_joint" type="fixed">
             <origin xyz="0 0 0" rpy="${-pi/2} 0 ${-pi/2}"/>
-            <parent link="${prefix}_depth_camera" />
+            <parent link="${prefix}_depth_camera_link" />
             <child link="${prefix}_depth_camera_optical_link" />
         </joint>
+        <link name="${prefix}_depth_camera_base_link" />
         <joint name="${prefix}_depth_camera_joint" type="fixed">
+            <origin xyz="0 0 ${height/2}" rpy="0 0 0"/>
+            <parent link="${prefix}_depth_camera_base_link" />
+            <child link="${prefix}_depth_camera_link" />
+        </joint>
+        <joint name="${prefix}_depth_camera_base_joint" type="fixed">
             <xacro:insert_block name="joint_origin" />
             <parent link="${parent}" />
-            <child link="${prefix}_depth_camera" />
+            <child link="${prefix}_depth_camera_base_link" />
             <axis xyz="0 1 0" />
         </joint>

Commit message: Switch to libgazebo_ros_camera.so for simulation, organize depth camera xacro

File: marvin_simulation/urdf/depth_camera.xacro (robot description, xacro)
@@ -3,4 +3,13 @@
     <xacro:macro name="depth_camera" params="prefix mass length width height parent:=base_link *joint_origin">
         <xacro:include filename="$(find marvin_simulation)/urdf/inertia.xacro"/>
+        <!-- Depth camera base link -->
+        <link name="${prefix}_depth_camera_base_link" />
+        <joint name="${prefix}_depth_camera_base_joint" type="fixed">
+            <xacro:insert_block name="joint_origin" />
+            <parent link="${parent}" />
+            <child link="${prefix}_depth_camera_base_link" />
+            <axis xyz="0 1 0" />
+        </joint>
+        <!-- Depth camera link -->
         <link name="${prefix}_depth_camera_link">
             <xacro:box_inertia mass="${mass}" length="${length}" width="${width}" height="${height}">
@@ -20,4 +29,10 @@
             </collision>
         </link>
+        <joint name="${prefix}_depth_camera_joint" type="fixed">
+            <origin xyz="0 0 ${height/2}" rpy="0 0 0"/>
+            <parent link="${prefix}_depth_camera_base_link" />
+            <child link="${prefix}_depth_camera_link" />
+        </joint>
+        <!-- Depth camera optical link -->
         <link name="${prefix}_depth_camera_optical_link" />
         <joint name="${prefix}_depth_camera_optical_joint" type="fixed">
@@ -26,61 +41,31 @@
             <child link="${prefix}_depth_camera_optical_link" />
         </joint>
-        <link name="${prefix}_depth_camera_base_link" />
-        <joint name="${prefix}_depth_camera_joint" type="fixed">
-            <origin xyz="0 0 ${height/2}" rpy="0 0 0"/>
-            <parent link="${prefix}_depth_camera_base_link" />
-            <child link="${prefix}_depth_camera_link" />
-        </joint>
-        <joint name="${prefix}_depth_camera_base_joint" type="fixed">
-            <xacro:insert_block name="joint_origin" />
-            <parent link="${parent}" />
-            <child link="${prefix}_depth_camera_base_link" />
-            <axis xyz="0 1 0" />
-        </joint>
-        <gazebo reference="${prefix}_depth_camera">
-            <material>Gazebo/Yellow</material>
+        <!-- Depth camera color -->
+        <gazebo reference="${prefix}_depth_camera_link">
+            <material>Gazebo/Black</material>
         </gazebo>
-        <gazebo reference="${prefix}_depth_camera">
-            <sensor type="depth" name="camera1">
-            <update_rate>15.0</update_rate>
-            <camera name="head">
-                <horizontal_fov>1.91986</horizontal_fov>
-                <image>
-                <width>2560</width>
-                <height>720</height>
-                <format>R8G8B8</format>
-                </image>
-                <clip>
-                <near>0.02</near>
-                <far>300</far>
-                </clip>
-            </camera>
-            <!-- change the plugin to a depth cam-->
-            <plugin name="${prefix}_depth_camera_plugin" filename="libgazebo_ros_openni_kinect.so">
-                <baseline>0.2</baseline>
-                <alwaysOn>true</alwaysOn>
-                <!-- Keep this zero, update_rate in the parent <sensor> tag
-                will control the frame rate. -->
-                <updateRate>0.0</updateRate>
-                <cameraName>camera_ir</cameraName>
-                <imageTopicName>/camera/color/image_raw</imageTopicName>
-                <cameraInfoTopicName>/camera/color/camera_info</cameraInfoTopicName>
-                <depthImageTopicName>/camera/depth/image_raw</depthImageTopicName>
-                <depthImageCameraInfoTopicName>/camera/depth/camera_info</depthImageCameraInfoTopicName>
-                <pointCloudTopicName>/camera/depth/points</pointCloudTopicName> <!-- /camera/depth/points -->
-                <frameName>camera_link_optical</frameName>
-                <pointCloudCutoff>0.3</pointCloudCutoff>
-                <pointCloudCutoffMax>20</pointCloudCutoffMax>
-                <distortionK1>0</distortionK1>
-                <distortionK2>0</distortionK2>
-                <distortionK3>0</distortionK3>
-                <distortionT1>0</distortionT1>
-                <distortionT2>0</distortionT2>
-                <CxPrime>0</CxPrime>
-                <Cx>0</Cx>
-                <Cy>0</Cy>
-                <focalLength>0</focalLength>
-                <hackBaseline>0</hackBaseline>
-            </plugin>
+        <!-- Depth camera plugin -->
+        <gazebo reference="${prefix}_depth_camera_link">
+            <sensor name="${prefix}_depth_camera" type="depth">
+                <update_rate>10.0</update_rate>
+                <visualize>true</visualize>
+                <always_on>true</always_on>
+                <camera>
+                    <horizontal_fov>1.91986</horizontal_fov>
+                    <image>
+                        <width>640</width>
+                        <height>480</height>
+                        <format>B8G8R8</format>
+                    </image>
+                    <clip>
+                        <near>0.05</near>
+                        <far>8.0</far>
+                    </clip>
+                </camera>
+                <plugin name="${prefix}_depth_camera_controller" filename="libgazebo_ros_camera.so">
+                    <frame_name>${prefix}_depth_camera_optical_link</frame_name>
+                    <min_depth>0.1</min_depth>
+                    <max_depth>100.0</max_depth>
+                </plugin>
             </sensor>
         </gazebo>
