Commit message: Format wheel.xacro to fit convention

File: marvin_simulation/urdf/wheel.xacro (robot description, xacro)
@@ -1,7 +1,8 @@
 <?xml version="1.0"?>
 <robot xmlns:xacro="http://ros.org/wiki/xacro" name="wheel">
-    <xacro:macro name="wheel" params="prefix mass radius width *joint_origin">
+    <xacro:macro name="wheel" params="prefix mass radius width parent:=base_link *joint_origin">
         <xacro:include filename="$(find marvin_simulation)/urdf/inertia.xacro"/>
-        <link name="${prefix}_wheel">
+        <!-- Wheel link -->
+        <link name="${prefix}_wheel_link">
             <xacro:cylinder_inertia mass="${mass}" radius="${radius}" height="${width}">
                 <origin xyz="0 0 0" rpy="0 0 0" />
@@ -28,4 +29,5 @@
             <dynamics damping="0.0001"/>
         </joint>
+        <!-- Wheel color & physics-->
         <gazebo reference="${prefix}_wheel">
             <material>Gazebo/Green</material>

Commit message: Fix wheel breaking change

File: marvin_simulation/urdf/wheel.xacro (robot description, xacro)
@@ -24,5 +24,5 @@
             <xacro:insert_block name="joint_origin" />
             <parent link="base_link" />
-            <child link="${prefix}_wheel" />
+            <child link="${prefix}_wheel_link" />
             <axis xyz="0 1 0" rpy="0 0 0" />
             <limit effort="1000" velocity="1000"/>
@@ -30,5 +30,5 @@
         </joint>
         <!-- Wheel color & physics-->
-        <gazebo reference="${prefix}_wheel">
+        <gazebo reference="${prefix}_wheel_link">
             <material>Gazebo/Green</material>
             <mu1 value="1.0"/>
