Commit message: #9 fix endoder position

File: marvin_simulation/urdf/marvin.xacro (robot description, xacro)
@@ -169,5 +169,5 @@
     <link name="encoders" />
 	<joint name="encoders_joint" type="fixed">
-		<origin xyz="0 0 ${wheel_radius}" rpy="0 0 0" />
+		<origin xyz="0 0 ${wheel_radius-chassis_z_offset}" rpy="0 0 0" />
 		<parent link="base_link" />
 		<child link="encoders" />

Commit message: Add proper camera dimensions and mass

File: marvin_simulation/urdf/marvin.xacro (robot description, xacro)
@@ -32,5 +32,8 @@
     <xacro:property name="lidar_height" value="${32.55*0.0254}"/>
     <!-- Camera Constants -->
-    <xacro:property name="camera_mass" value="0.1"/>
+    <xacro:property name="camera_mass" value="0.230"/>
+    <xacro:property name="camera_length" value="0.04310"/>
+    <xacro:property name="camera_width" value="0.17525"/>
+    <xacro:property name="camera_height" value="0.03025"/>
     <xacro:property name="camera_angle" value="${10 * 0.01745327777}"/>
     <xacro:property name="camera_x_offset" value="${(4+2.66916)*0.0254}"/>
@@ -134,5 +137,5 @@
     <!-- Sim Camera -->
 	<xacro:include filename="$(find marvin_simulation)/urdf/depth_camera.xacro" />
-	<xacro:depth_camera prefix="zed" mass="${camera_mass}" length = "${1.5*0.0254}" width="${6.75*0.0254}" height="${1*0.0254}" parent="base_link">
+	<xacro:depth_camera prefix="zed" mass="${camera_mass}" length = "${camera_length}" width="${camera_width}" height="${camera_height}" parent="base_link">
 		<origin xyz="${camera_x_offset} 0 ${camera_z_offset}" rpy="0 ${camera_angle} 0" />
 	</xacro:depth_camera>
@@ -193,5 +196,5 @@
 		<material>Gazebo/Purple</material>
 	</gazebo>
-    <!-- Motor, Camera and IMU Simulation -->
+    <!-- Motor and IMU Simulation -->
 	<xacro:include filename="$(find marvin_simulation)/urdf/marvin.gazebo" />
 </robot>

Commit message: Move caster into independent block

File: marvin_simulation/urdf/marvin.xacro (robot description, xacro)
@@ -98,33 +98,8 @@
     </joint>
     <!-- Caster -->
-    <link name="caster">
-        <visual name="caster_visual">
-            <geometry>
-                <sphere radius="${caster_radius}" />
-            </geometry>
-        </visual>
-        <collision name='caster_collision'>
-			<origin xyz="0 0 0" rpy=" 0 0 0"/>
-			<geometry>
-				<sphere radius="${caster_radius}"/>
-			</geometry>
-			<surface>
-				<friction>
-				<ode>
-					<mu>0.0</mu>
-					<mu2>0.0</mu2>
-				</ode>
-				</friction>
-			</surface>
-		</collision>
-        <xacro:sphere_inertia mass="${caster_mass}" radius="${caster_radius}">
-            <origin xyz="0 0 0" rpy="0 0 0" />
-        </xacro:sphere_inertia>
-    </link>
-    <joint name="caster_joint" type="fixed">
+    <xacro:include filename="$(find marvin_simulation)/urdf/caster.xacro"/>
+	<xacro:caster prefix="back" mass="${caster_mass}" radius="${caster_radius}">
         <origin xyz="${caster_x_offset} 0 ${caster_radius-chassis_z_offset}" rpy="0 0 0" />
-        <parent link="base_link" />
-        <child link="caster" />
-    </joint>
+	</xacro:caster>
     <!-- Wheels -->
     <xacro:include filename="$(find marvin_simulation)/urdf/wheel.xacro"/>
@@ -190,7 +165,4 @@
 		<material>Gazebo/Blue</material>
 	</gazebo>
-	<gazebo reference="caster_visual">
-		<material>Gazebo/Green</material>
-	</gazebo>
 	<gazebo reference="imu_visual">
 		<material>Gazebo/Purple</material>

Commit message: Move IMU to independent block

File: marvin_simulation/urdf/marvin.xacro (robot description, xacro)
@@ -121,27 +121,8 @@
 	</xacro:VLP-16>
 	<!-- IMU -->
-	<link name="imu_link">
-		<visual name="imu_visual">
-			<origin xyz="0 0 0" rpy="0 0 0" />
-			<geometry>
-				<box size="0.05 0.03 0.01" />
-			</geometry>
-		</visual>
-        <collision name="imu_collision">
-            <origin xyz="0 0 0" rpy="0 0 0" />
-            <geometry>
-                <box size="${imu_length} ${imu_width} ${imu_height}" />
-            </geometry>
-        </collision>
-        <xacro:box_inertia mass="${imu_mass}" length="${imu_length}" width="${imu_width}" height="${imu_height}">
-            <origin xyz="0 0 0" rpy="0 0 0" />
-        </xacro:box_inertia>
-	</link>
-	<joint name="imu_joint" type="fixed">
-		<origin xyz="${-chassis_tower_length / 2 - chassis_electrical_length/2+0.005} 0 ${chassis_electrical_height}" rpy="0 0 0" />
-		<parent link="base_link" />
-		<child link="imu_link" />
-		<axis xyz="0 1 0" />
-	</joint>
+    <xacro:include filename="$(find marvin_simulation)/urdf/imu.xacro" />
+    <xacro:imu prefix="robot" mass="${imu_mass}" length="${imu_length}" width="${imu_width}" height="${imu_height}">
+		<origin xyz="${-chassis_tower_length / 2 - chassis_electrical_length/2} 0 ${chassis_electrical_height}" rpy="0 0 0" />
+    </xacro:imu>
     <!-- Encoders -->
     <link name="encoders" />
@@ -165,8 +146,5 @@
 		<material>Gazebo/Blue</material>
 	</gazebo>
-	<gazebo reference="imu_visual">
-		<material>Gazebo/Purple</material>
-	</gazebo>
-    <!-- Motor and IMU Simulation -->
+    <!-- Motor Simulation -->
 	<xacro:include filename="$(find marvin_simulation)/urdf/marvin.gazebo" />
 </robot>

Commit message: Move diff drive controller to xacro, fix color bug and encoder typo

File: marvin_simulation/urdf/marvin.xacro (robot description, xacro)
@@ -47,5 +47,8 @@
 	<!-- Chassis -->
 	<link name="base_link">
-		<visual name="chassis_tower_visual">
+        <xacro:box_inertia mass="${chassis_mass}" length="${chassis_length}" width="${chassis_width}" height="${chassis_height}">
+            <origin xyz="${com_x} ${com_y} ${com_z}" rpy="0 0 0" />
+		</xacro:box_inertia>
+		<visual> <!-- Chassis Tower -->
 			<origin xyz="0 0 ${chassis_tower_height / 2}" rpy="0 0 0" />
 			<geometry>
@@ -53,5 +56,5 @@
 			</geometry>
 		</visual>
-        <visual name="chassis_payload_visual">
+        <visual> <!-- Chassis Payload -->
             <origin xyz="${chassis_tower_length / 2 + chassis_payload_length / 2} 0 ${chassis_payload_height / 2}" rpy="0 0 0" />
             <geometry>
@@ -59,5 +62,5 @@
             </geometry>
         </visual>
-        <visual name="chassis_electrical_visual">
+        <visual> <!-- Chassis Electrical -->
             <origin xyz="${-chassis_tower_length / 2 - chassis_electrical_length / 2} 0 ${chassis_electrical_height / 2}" rpy="0 0 0" />
             <geometry>
@@ -65,5 +68,5 @@
             </geometry>
         </visual>
-        <visual name="chassis_caster_visual">
+        <visual> <!-- Chassis Caster -->
             <origin xyz="${-chassis_tower_length / 2 - chassis_electrical_length - chassis_caster_length / 2}
                          0
@@ -74,5 +77,5 @@
             </geometry>
         </visual>
-		<collision name="chassis_collision">
+		<collision>
 			<origin xyz="${chassis_tower_length / 2 + chassis_payload_length - chassis_length / 2}
                          0
@@ -83,8 +86,9 @@
 			</geometry>
 		</collision>
-        <xacro:box_inertia mass="${chassis_mass}" length="${chassis_length}" width="${chassis_width}" height="${chassis_height}">
-            <origin xyz="${com_x} ${com_y} ${com_z}" rpy="0 0 0" />
-		</xacro:box_inertia>
 	</link>
+    <gazebo reference="base_link">
+        <material>Gazebo/Blue</material>
+    </gazebo>
+    <!-- Footprint -->
     <link name="base_footprint">
         <xacro:box_inertia mass="0" length="0" width="0" height="0">
@@ -110,5 +114,5 @@
 		<origin xyz="0 ${track_width/2} ${wheel_radius-chassis_z_offset}" rpy="0 0 0" />
 	</xacro:wheel>
-    <!-- Sim Camera -->
+    <!-- Camera -->
 	<xacro:include filename="$(find marvin_simulation)/urdf/depth_camera.xacro" />
 	<xacro:depth_camera prefix="zed" mass="${camera_mass}" length = "${camera_length}" width="${camera_width}" height="${camera_height}" parent="base_link">
@@ -125,26 +129,34 @@
 		<origin xyz="${-chassis_tower_length / 2 - chassis_electrical_length/2} 0 ${chassis_electrical_height}" rpy="0 0 0" />
     </xacro:imu>
-    <!-- Encoders -->
-    <link name="encoders" />
-	<joint name="encoders_joint" type="fixed">
+    <!-- Encoder -->
+    <link name="encoder" />
+	<joint name="encoder_joint" type="fixed">
 		<origin xyz="0 0 ${wheel_radius-chassis_z_offset}" rpy="0 0 0" />
 		<parent link="base_link" />
-		<child link="encoders" />
+		<child link="encoder" />
 		<axis xyz="0 1 0" />
 	</joint>
-    <!-- Color of bot -->
-	<gazebo reference="chassis_tower_visual">
-		<material>Gazebo/Blue</material>
+    <!-- Drivetrain Simulation -->
+	<gazebo>
+		<plugin name="differential_drive_controller" filename="libgazebo_ros_diff_drive.so">
+			<update_rate>100.0</update_rate>
+			<robot_base_frame>base_link</robot_base_frame>
+			<command_topic>cmd_vel</command_topic>
+			<left_joint>left_wheel_joint</left_joint>
+			<right_joint>right_wheel_joint</right_joint>
+			<wheel_separation>${track_width}</wheel_separation>
+			<wheel_diameter>${2 * wheel_radius}</wheel_diameter>
+			<publish_tf>true</publish_tf>
+			<publish_wheel_tf>true</publish_wheel_tf>
+			<max_wheel_acceleration>1.8</max_wheel_acceleration>
+			<max_wheel_torque>30</max_wheel_torque>
+			<odometrySource>encoder</odometrySource>
+			<odometry_topic>odom</odometry_topic>
+			<odometry_frame>odom</odometry_frame>
+			<publish_odom>true</publish_odom>
+			<publish_odom_tf>true</publish_odom_tf>
+			<legacy_mode>false</legacy_mode>
+			<ros_debug_level>na</ros_debug_level>
+		</plugin>
 	</gazebo>
-	<gazebo reference="chassis_payload_visual">
-		<material>Gazebo/Blue</material>
-	</gazebo>
-	<gazebo reference="chassis_electrical_visual">
-		<material>Gazebo/Blue</material>
-	</gazebo>
-	<gazebo reference="chassis_caster_visual">
-		<material>Gazebo/Blue</material>
-	</gazebo>
-    <!-- Motor Simulation -->
-	<xacro:include filename="$(find marvin_simulation)/urdf/marvin.gazebo" />
 </robot>

Commit message: Move chassis, constants and plugins to independent file

File: marvin_simulation/urdf/marvin.xacro (robot description, xacro)
@@ -1,99 +1,9 @@
 <?xml version='1.0'?>
 <robot name="marvin" xmlns:xacro="http://www.ros.org/wiki/xacro">
-	<!-- Chassis Constants -->
-    <xacro:property name="chassis_length" value="${45.5*0.0254}" />
-    <xacro:property name="chassis_width" value="${24*0.0254}" />
-    <xacro:property name="chassis_height" value="${22*0.0254}" />
-    <xacro:property name="chassis_z_offset" value="${4.375*0.0254}" />
-    <xacro:property name="chassis_tower_length" value="${8*0.0254}" />
-    <xacro:property name="chassis_tower_height" value="${31*0.0254}" />
-    <xacro:property name="chassis_payload_length" value="${14.25*0.0254}" />
-    <xacro:property name="chassis_payload_height" value="${8*0.0254}" />
-    <xacro:property name="chassis_electrical_length" value="${15.25*0.0254}" />
-    <xacro:property name="chassis_electrical_height" value="${22*0.0254}" />
-    <xacro:property name="chassis_caster_length" value="${8*0.0254}" />
-    <xacro:property name="chassis_caster_height" value="${2.25*0.0254}" />
-    <xacro:property name="chassis_caster_z_offset" value="${2*0.0254}" />
-    <!-- Chassis Inertial Constants -->
-    <xacro:property name="chassis_mass" value="29.9371" />
-    <xacro:property name="com_x" value="${-4.0*0.0254}" />
-    <xacro:property name="com_y" value="0.0" />
-    <xacro:property name="com_z" value="${6.1875*0.0254-chassis_z_offset}" />
-	<!-- Caster Constants -->
-    <xacro:property name="caster_x_offset" value="${-24.625*0.0254}" />
-    <xacro:property name="caster_radius" value="${3.5*0.0254}" />
-    <xacro:property name="caster_mass" value="0.1" />
-	<!-- Wheel Constants -->
-    <xacro:property name="wheel_radius" value="${6.1875*0.0254}" />
-    <xacro:property name="wheel_width" value="${4*0.0254}" />
-    <xacro:property name="wheel_mass" value="5" />
-    <xacro:property name="track_width" value="${31*0.0254}" />
-    <!-- Lidar Constants -->
-    <xacro:property name="lidar_height" value="${32.55*0.0254}"/>
-    <!-- Camera Constants -->
-    <xacro:property name="camera_mass" value="0.230"/>
-    <xacro:property name="camera_length" value="0.04310"/>
-    <xacro:property name="camera_width" value="0.17525"/>
-    <xacro:property name="camera_height" value="0.03025"/>
-    <xacro:property name="camera_angle" value="${10 * 0.01745327777}"/>
-    <xacro:property name="camera_x_offset" value="${(4+2.66916)*0.0254}"/>
-    <xacro:property name="camera_z_offset" value="${(31-1.80395)*0.0254}"/>
-    <!-- IMU Constants -->
-    <xacro:property name="imu_mass" value="0.025"/>
-    <xacro:property name="imu_length" value="0.05"/>
-    <xacro:property name="imu_width" value="0.03"/>
-    <xacro:property name="imu_height" value="0.01"/>
-	<xacro:include filename="$(find marvin_simulation)/urdf/inertia.xacro" />
-	<!-- Chassis -->
-	<link name="base_link">
-        <xacro:box_inertia mass="${chassis_mass}" length="${chassis_length}" width="${chassis_width}" height="${chassis_height}">
-            <origin xyz="${com_x} ${com_y} ${com_z}" rpy="0 0 0" />
-		</xacro:box_inertia>
-		<visual> <!-- Chassis Tower -->
-			<origin xyz="0 0 ${chassis_tower_height / 2}" rpy="0 0 0" />
-			<geometry>
-				<box size="${chassis_tower_length} ${chassis_width} ${chassis_tower_height}" />
-			</geometry>
-		</visual>
-        <visual> <!-- Chassis Payload -->
-            <origin xyz="${chassis_tower_length / 2 + chassis_payload_length / 2} 0 ${chassis_payload_height / 2}" rpy="0 0 0" />
-            <geometry>
-                <box size="${chassis_payload_length} ${chassis_width} ${chassis_payload_height}" />
-            </geometry>
-        </visual>
-        <visual> <!-- Chassis Electrical -->
-            <origin xyz="${-chassis_tower_length / 2 - chassis_electrical_length / 2} 0 ${chassis_electrical_height / 2}" rpy="0 0 0" />
-            <geometry>
-                <box size="${chassis_electrical_length} ${chassis_width} ${chassis_electrical_height}" />
-            </geometry>
-        </visual>
-        <visual> <!-- Chassis Caster -->
-            <origin xyz="${-chassis_tower_length / 2 - chassis_electrical_length - chassis_caster_length / 2}
-                         0
-                         ${chassis_caster_height / 2 + chassis_caster_z_offset}"
-                         rpy="0 0 0" />
-            <geometry>
-                <box size="${chassis_caster_length} ${chassis_width} ${chassis_caster_height}" />
-            </geometry>
-        </visual>
-		<collision>
-			<origin xyz="${chassis_tower_length / 2 + chassis_payload_length - chassis_length / 2}
-                         0
-                         ${chassis_tower_height / 2}"
-                    rpy="0 0 0" />
-			<geometry>
-				<box size="${chassis_length} ${chassis_width} ${chassis_tower_height}" />
-			</geometry>
-		</collision>
-	</link>
-    <gazebo reference="base_link">
-        <material>Gazebo/Blue</material>
-    </gazebo>
+    <xacro:include filename="$(find marvin_simulation)/urdf/constants.xacro"/>
+	<!-- Base_link -->
+    <link name="base_link" />
     <!-- Footprint -->
-    <link name="base_footprint">
-        <xacro:box_inertia mass="0" length="0" width="0" height="0">
-            <origin xyz="0 0 0" rpy="0 0 0" />
-        </xacro:box_inertia>
-    </link>
+    <link name="base_footprint" />
     <joint name="base_joint" type="fixed">
         <origin xyz="0 0 ${-chassis_z_offset}" rpy="0 0 0" />
@@ -101,4 +11,6 @@
         <child link="base_footprint" />
     </joint>
+    <!-- Chassis -->
+    <xacro:include filename="$(find marvin_simulation)/urdf/chassis.xacro"/>
     <!-- Caster -->
     <xacro:include filename="$(find marvin_simulation)/urdf/caster.xacro"/>
@@ -137,26 +49,5 @@
 		<axis xyz="0 1 0" />
 	</joint>
-    <!-- Drivetrain Simulation -->
-	<gazebo>
-		<plugin name="differential_drive_controller" filename="libgazebo_ros_diff_drive.so">
-			<update_rate>100.0</update_rate>
-			<robot_base_frame>base_link</robot_base_frame>
-			<command_topic>cmd_vel</command_topic>
-			<left_joint>left_wheel_joint</left_joint>
-			<right_joint>right_wheel_joint</right_joint>
-			<wheel_separation>${track_width}</wheel_separation>
-			<wheel_diameter>${2 * wheel_radius}</wheel_diameter>
-			<publish_tf>true</publish_tf>
-			<publish_wheel_tf>true</publish_wheel_tf>
-			<max_wheel_acceleration>1.8</max_wheel_acceleration>
-			<max_wheel_torque>30</max_wheel_torque>
-			<odometrySource>encoder</odometrySource>
-			<odometry_topic>odom</odometry_topic>
-			<odometry_frame>odom</odometry_frame>
-			<publish_odom>true</publish_odom>
-			<publish_odom_tf>true</publish_odom_tf>
-			<legacy_mode>false</legacy_mode>
-			<ros_debug_level>na</ros_debug_level>
-		</plugin>
-	</gazebo>
+    <!-- Gazebo plugins -->
+    <xacro:include filename="$(find marvin_simulation)/urdf/plugins.xacro"/>
 </robot>
