Commit message: Update caster xacro to have proper color

File: marvin_simulation/urdf/caster.xacro (robot description, xacro)
@@ -4,5 +4,5 @@
         <xacro:include filename="$(find marvin_simulation)/urdf/inertia.xacro"/>
         <!-- Caster link -->
-        <link name="${prefix}_caster">
+        <link name="${prefix}_caster_link">
             <xacro:sphere_inertia mass="${mass}" radius="${radius}">
                 <origin xyz="0 0 0" rpy="0 0 0" />
@@ -28,11 +28,11 @@
             </collision>
         </link>
-        <joint name="caster_joint" type="fixed">
+        <joint name="${prefix}_caster_joint" type="fixed">
             <xacro:insert_block name="joint_origin" />
             <parent link="${parent}" />
-            <child link="${prefix}_caster" />
+            <child link="${prefix}_caster_link" />
         </joint>
         <!-- Caster color -->
-        <gazebo reference="caster_visual">
+        <gazebo reference="${prefix}_caster_link">
 		    <material>Gazebo/Green</material>
 	    </gazebo>

Commit message: Make blocks take name and not prefix

File: marvin_simulation/urdf/caster.xacro (robot description, xacro)
@@ -1,8 +1,8 @@
 <?xml version="1.0"?>
 <robot xmlns:xacro="http://ros.org/wiki/xacro" name="caster">
-    <xacro:macro name="caster" params="prefix mass radius parent:=base_link *joint_origin">
+    <xacro:macro name="caster" params="name mass radius parent:=base_link *joint_origin">
         <xacro:include filename="$(find marvin_simulation)/urdf/inertia.xacro"/>
         <!-- Caster link -->
-        <link name="${prefix}_caster_link">
+        <link name="${name}_link">
             <xacro:sphere_inertia mass="${mass}" radius="${radius}">
                 <origin xyz="0 0 0" rpy="0 0 0" />
@@ -28,11 +28,11 @@
             </collision>
         </link>
-        <joint name="${prefix}_caster_joint" type="fixed">
+        <joint name="${name}_joint" type="fixed">
             <xacro:insert_block name="joint_origin" />
             <parent link="${parent}" />
-            <child link="${prefix}_caster_link" />
+            <child link="${name}_link" />
         </joint>
         <!-- Caster color -->
-        <gazebo reference="${prefix}_caster_link">
+        <gazebo reference="${name}_link">
 		    <material>Gazebo/Green</material>
 	    </gazebo>

File: marvin_simulation/urdf/depth_camera.xacro (robot description, xacro)
@@ -1,16 +1,16 @@
 <?xml version="1.0"?>
 <robot xmlns:xacro="http://ros.org/wiki/xacro" name="depth_camera">
-    <xacro:macro name="depth_camera" params="prefix mass length width height parent:=base_link *joint_origin">
+    <xacro:macro name="depth_camera" params="name mass length width height parent:=base_link *joint_origin">
         <xacro:include filename="$(find marvin_simulation)/urdf/inertia.xacro"/>
         <!-- Depth camera base link -->
-        <link name="${prefix}_depth_camera_base_link" />
-        <joint name="${prefix}_depth_camera_base_joint" type="fixed">
+        <link name="${name}_base_link" />
+        <joint name="${name}_base_joint" type="fixed">
             <xacro:insert_block name="joint_origin" />
             <parent link="${parent}" />
-            <child link="${prefix}_depth_camera_base_link" />
+            <child link="${name}_base_link" />
             <axis xyz="0 1 0" />
         </joint>
         <!-- Depth camera link -->
-        <link name="${prefix}_depth_camera_link">
+        <link name="${name}_link">
             <xacro:box_inertia mass="${mass}" length="${length}" width="${width}" height="${height}">
                 <origin xyz="0 0 0" rpy="0 0 0" />
@@ -29,23 +29,23 @@
             </collision>
         </link>
-        <joint name="${prefix}_depth_camera_joint" type="fixed">
+        <joint name="${name}_joint" type="fixed">
             <origin xyz="0 0 ${height/2}" rpy="0 0 0"/>
-            <parent link="${prefix}_depth_camera_base_link" />
-            <child link="${prefix}_depth_camera_link" />
+            <parent link="${name}_base_link" />
+            <child link="${name}_link" />
         </joint>
         <!-- Depth camera optical link -->
-        <link name="${prefix}_depth_camera_optical_link" />
-        <joint name="${prefix}_depth_camera_optical_joint" type="fixed">
+        <link name="${name}_optical_link" />
+        <joint name="${name}_optical_joint" type="fixed">
             <origin xyz="0 0 0" rpy="${-pi/2} 0 ${-pi/2}"/>
-            <parent link="${prefix}_depth_camera_link" />
-            <child link="${prefix}_depth_camera_optical_link" />
+            <parent link="${name}_link" />
+            <child link="${name}_optical_link" />
         </joint>
         <!-- Depth camera color -->
-        <gazebo reference="${prefix}_depth_camera_link">
+        <gazebo reference="${name}_link">
             <material>Gazebo/Black</material>
         </gazebo>
         <!-- Depth camera plugin -->
-        <gazebo reference="${prefix}_depth_camera_link">
-            <sensor name="${prefix}_depth_camera" type="depth">
+        <gazebo reference="${name}_link">
+            <sensor name="${name}" type="depth">
                 <update_rate>15.0</update_rate>
                 <visualize>true</visualize>
@@ -63,6 +63,6 @@
                     </clip>
                 </camera>
-                <plugin name="${prefix}_depth_camera_controller" filename="libgazebo_ros_camera.so">
-                    <frame_name>${prefix}_depth_camera_optical_link</frame_name>
+                <plugin name="${name}_controller" filename="libgazebo_ros_camera.so">
+                    <frame_name>${name}_optical_link</frame_name>
                     <min_depth>0</min_depth>
                     <max_depth>100</max_depth>

File: marvin_simulation/urdf/imu.xacro (robot description, xacro)
@@ -1,16 +1,16 @@
 <?xml version="1.0"?>
 <robot xmlns:xacro="http://ros.org/wiki/xacro" name="caster">
-    <xacro:macro name="imu" params="prefix mass length width height parent:=base_link *joint_origin">
+    <xacro:macro name="imu" params="name mass length width height parent:=base_link *joint_origin">
         <xacro:include filename="$(find marvin_simulation)/urdf/inertia.xacro"/>
         <!-- imu base link -->
-        <link name="${prefix}_imu_base_link" />
-        <joint name="${prefix}_imu_base_joint" type="fixed">
+        <link name="${name}_base_link" />
+        <joint name="${name}_base_joint" type="fixed">
             <xacro:insert_block name="joint_origin" />
             <parent link="${parent}" />
-            <child link="${prefix}_imu_base_link" />
+            <child link="${name}_base_link" />
             <axis xyz="0 1 0" />
         </joint>
         <!-- imu link -->
-        <link name="${prefix}_imu_link">
+        <link name="${name}_link">
 		    <xacro:box_inertia mass="${mass}" length="${length}" width="${width}" height="${height}">
                 <origin xyz="0 0 0" rpy="0 0 0" />
@@ -29,17 +29,17 @@
             </collision>
         </link>
-        <joint name="${prefix}_imu_joint" type="fixed">
+        <joint name="${name}_joint" type="fixed">
             <origin xyz="0 0 ${height/2}" rpy="0 0 0"/>
-            <parent link="${prefix}_imu_base_link" />
-            <child link="${prefix}_imu_link" />
+            <parent link="${name}_base_link" />
+            <child link="${name}_link" />
         </joint>
         <!-- imu color -->
-        <gazebo reference="${prefix}_imu_link">
+        <gazebo reference="${name}_link">
             <material>Gazebo/Purple</material>
         </gazebo>
         <!-- imu plugin -->
-        <gazebo reference="${prefix}_imu_link">
+        <gazebo reference="${name}_link">
             <gravity>true</gravity>
-            <sensor name="${prefix}_imu" type="imu">
+            <sensor name="${name}" type="imu">
                 <always_on>true</always_on>
                 <update_rate>100.0</update_rate>
@@ -47,12 +47,12 @@
                 <topic>__default_topic__</topic>
                 <pose>0 0 0 0 0 0</pose>
-                <plugin name="${prefix}_imu_controller" filename="libgazebo_ros_imu_sensor.so">
+                <plugin name="${name}_controller" filename="libgazebo_ros_sensor.so">
                     <topicName>imu</topicName>
-                    <bodyName>${prefix}_imu_link</bodyName>
+                    <bodyName>${name}_link</bodyName>
                     <updateRateHZ>100.0</updateRateHZ>
                     <gaussianNoise>0.0</gaussianNoise>
                     <xyzOffset>0 0 0</xyzOffset>
                     <rpyOffset>0 0 0</rpyOffset>
-                    <frameName>${prefix}_imu_link</frameName>
+                    <frameName>${name}_link</frameName>
                     <initialOrientationAsReference>false</initialOrientationAsReference>
                 </plugin>

File: marvin_simulation/urdf/marvin.xacro (robot description, xacro)
@@ -15,18 +15,18 @@
     <!-- Caster -->
     <xacro:include filename="$(find marvin_simulation)/urdf/caster.xacro"/>
-	<xacro:caster prefix="back" mass="${caster_mass}" radius="${caster_radius}">
+	<xacro:caster name="caster" mass="${caster_mass}" radius="${caster_radius}">
         <origin xyz="${caster_x_offset} 0 ${caster_radius-chassis_z_offset}" rpy="0 0 0" />
 	</xacro:caster>
     <!-- Wheels -->
     <xacro:include filename="$(find marvin_simulation)/urdf/wheel.xacro"/>
-	<xacro:wheel prefix="right" mass="${wheel_mass}" radius="${wheel_radius}" width="${wheel_width}">
+	<xacro:wheel name="right_wheel" mass="${wheel_mass}" radius="${wheel_radius}" width="${wheel_width}">
 		<origin xyz="0 -${track_width / 2} ${wheel_radius-chassis_z_offset}" rpy="0 0 0" />
 	</xacro:wheel>
-	<xacro:wheel prefix="left" mass="${wheel_mass}" radius="${wheel_radius}" width="${wheel_width}">
+	<xacro:wheel name="left_wheel" mass="${wheel_mass}" radius="${wheel_radius}" width="${wheel_width}">
 		<origin xyz="0 ${track_width/2} ${wheel_radius-chassis_z_offset}" rpy="0 0 0" />
 	</xacro:wheel>
     <!-- Camera -->
 	<xacro:include filename="$(find marvin_simulation)/urdf/depth_camera.xacro" />
-	<xacro:depth_camera prefix="zed" mass="${camera_mass}" length = "${camera_length}" width="${camera_width}" height="${camera_height}" parent="base_link">
+	<xacro:depth_camera name="zed" mass="${camera_mass}" length = "${camera_length}" width="${camera_width}" height="${camera_height}" parent="base_link">
 		<origin xyz="${camera_x_offset} 0 ${camera_z_offset}" rpy="0 ${camera_angle} 0" />
 	</xacro:depth_camera>
@@ -38,5 +38,5 @@
 	<!-- IMU -->
     <xacro:include filename="$(find marvin_simulation)/urdf/imu.xacro" />
-    <xacro:imu prefix="robot" mass="${imu_mass}" length="${imu_length}" width="${imu_width}" height="${imu_height}">
+    <xacro:imu name="imu" mass="${imu_mass}" length="${imu_length}" width="${imu_width}" height="${imu_height}">
 		<origin xyz="${-chassis_tower_length / 2 - chassis_electrical_length/2} 0 ${chassis_electrical_height}" rpy="0 0 0" />
     </xacro:imu>

File: marvin_simulation/urdf/wheel.xacro (robot description, xacro)
@@ -1,8 +1,8 @@
 <?xml version="1.0"?>
 <robot xmlns:xacro="http://ros.org/wiki/xacro" name="wheel">
-    <xacro:macro name="wheel" params="prefix mass radius width parent:=base_link *joint_origin">
+    <xacro:macro name="wheel" params="name mass radius width parent:=base_link *joint_origin">
         <xacro:include filename="$(find marvin_simulation)/urdf/inertia.xacro"/>
         <!-- Wheel link -->
-        <link name="${prefix}_wheel_link">
+        <link name="${name}_link">
             <xacro:cylinder_inertia mass="${mass}" radius="${radius}" height="${width}">
                 <origin xyz="0 0 0" rpy="0 0 0" />
@@ -21,8 +21,8 @@
             </collision>
         </link>
-        <joint type="continuous" name="${prefix}_wheel_joint">
+        <joint type="continuous" name="${name}_joint">
             <xacro:insert_block name="joint_origin" />
             <parent link="base_link" />
-            <child link="${prefix}_wheel_link" />
+            <child link="${name}_link" />
             <axis xyz="0 1 0" rpy="0 0 0" />
             <limit effort="1000" velocity="1000"/>
@@ -30,5 +30,5 @@
         </joint>
         <!-- Wheel color & physics-->
-        <gazebo reference="${prefix}_wheel_link">
+        <gazebo reference="${name}_link">
             <material>Gazebo/Green</material>
             <mu1 value="1.0"/>
