Commit message: Rename lidar constant for convention

File: marvin_simulation/urdf/constants.xacro (robot description, xacro)
@@ -27,5 +27,5 @@
     <xacro:property name="wheel_z_offset" value="${1.8125*0.0254}"/>
     <!-- Lidar Constants -->
-    <xacro:property name="lidar_height" value="${32.55*0.0254}"/>
+    <xacro:property name="lidar_z_offset" value="${32.55*0.0254}"/>
     <!-- Camera Constants -->
     <xacro:property name="camera_angle" value="${10 * 0.01745327777}"/>

File: marvin_simulation/urdf/marvin.xacro (robot description, xacro)
@@ -35,5 +35,5 @@
     <xacro:include filename="$(find velodyne_description)/urdf/VLP-16.urdf.xacro" />
 	<xacro:VLP-16 parent="base_link" name="velodyne" topic="/velodyne_points" hz="20" samples="440" gpu="true">
-		<origin xyz="0 0 ${lidar_height}" rpy="0 0 0" />
+		<origin xyz="0 0 ${lidar_z_offset}" rpy="0 0 0" />
 	</xacro:VLP-16>
 	<!-- IMU -->
