Commit message: Make IMU dimension specific

File: common_xacro/urdf/sensor/imu.xacro (robot description, xacro)
@@ -6,26 +6,27 @@
 <!-- Plugin: libgazebo_ros_imu_sensor.so -->
 <!-- Param name: the name of the IMU. Published topic is /{name}_controller/out -->
-<!-- Param mass: mass of the IMU -->
-<!-- Param length: length of the IMU -->
-<!-- Param width: width of the IMU -->
-<!-- Param height: height of the IMU -->
 <!-- Param parent: name of the parent link, defaulted to base_link -->
 <!-- Param joint_origin: location of the IMU relative to parent link -->
 <robot xmlns:xacro="http://ros.org/wiki/xacro" name="caster">
-    <xacro:macro name="imu" params="name mass length width height parent:=base_link *joint_origin">
+    <xacro:macro name="imu" params="name parent:=base_link *joint_origin">
         <!-- Includes -->
         <xacro:include filename="$(find common_xacro)/urdf/physics/inertia.xacro"/>
+        <!-- Constants -->
+        <xacro:property name="mass" value="0.025"/>
+        <xacro:property name="length" value="0.05"/>
+        <xacro:property name="width" value="0.03"/>
+        <xacro:property name="height" value="0.01"/>
         <!-- Imu base link -->
-        <link name="${name}_base_link" />
+        <link name="${name}_base_link"/>
         <joint name="${name}_base_joint" type="fixed">
-            <xacro:insert_block name="joint_origin" />
-            <parent link="${parent}" />
-            <child link="${name}_base_link" />
-            <axis xyz="0 1 0" />
+            <xacro:insert_block name="joint_origin"/>
+            <parent link="${parent}"/>
+            <child link="${name}_base_link"/>
+            <axis xyz="0 1 0"/>
         </joint>
         <!-- Imu link -->
         <link name="${name}_link">
 		    <xacro:box_inertia mass="${mass}" length="${length}" width="${width}" height="${height}">
-                <origin xyz="0 0 0" rpy="0 0 0" />
+                <origin xyz="0 0 0" rpy="0 0 0"/>
             </xacro:box_inertia>
             <visual>
@@ -44,6 +45,6 @@
         <joint name="${name}_joint" type="fixed">
             <origin xyz="0 0 ${height/2}" rpy="0 0 0"/>
-            <parent link="${name}_base_link" />
-            <child link="${name}_link" />
+            <parent link="${name}_base_link"/>
+            <child link="${name}_link"/>
         </joint>
         <!-- Imu color -->

File: marvin_simulation/urdf/constants.xacro (robot description, xacro)
@@ -2,31 +2,31 @@
 <robot xmlns:xacro="http://ros.org/wiki/xacro" name="constants">
     <!-- Chassis Constants -->
-    <xacro:property name="chassis_length" value="${45.5*0.0254}" />
-    <xacro:property name="chassis_width" value="${24*0.0254}" />
-    <xacro:property name="chassis_height" value="${22*0.0254}" />
-    <xacro:property name="chassis_z_offset" value="${4.375*0.0254}" />
-    <xacro:property name="chassis_tower_length" value="${8*0.0254}" />
-    <xacro:property name="chassis_tower_height" value="${31*0.0254}" />
-    <xacro:property name="chassis_payload_length" value="${14.25*0.0254}" />
-    <xacro:property name="chassis_payload_height" value="${8*0.0254}" />
-    <xacro:property name="chassis_electrical_length" value="${15.25*0.0254}" />
-    <xacro:property name="chassis_electrical_height" value="${22*0.0254}" />
-    <xacro:property name="chassis_caster_length" value="${8*0.0254}" />
-    <xacro:property name="chassis_caster_height" value="${2.25*0.0254}" />
-    <xacro:property name="chassis_caster_z_offset" value="${2*0.0254}" />
+    <xacro:property name="chassis_length" value="${45.5*0.0254}"/>
+    <xacro:property name="chassis_width" value="${24*0.0254}"/>
+    <xacro:property name="chassis_height" value="${22*0.0254}"/>
+    <xacro:property name="chassis_z_offset" value="${4.375*0.0254}"/>
+    <xacro:property name="chassis_tower_length" value="${8*0.0254}"/>
+    <xacro:property name="chassis_tower_height" value="${31*0.0254}"/>
+    <xacro:property name="chassis_payload_length" value="${14.25*0.0254}"/>
+    <xacro:property name="chassis_payload_height" value="${8*0.0254}"/>
+    <xacro:property name="chassis_electrical_length" value="${15.25*0.0254}"/>
+    <xacro:property name="chassis_electrical_height" value="${22*0.0254}"/>
+    <xacro:property name="chassis_caster_length" value="${8*0.0254}"/>
+    <xacro:property name="chassis_caster_height" value="${2.25*0.0254}"/>
+    <xacro:property name="chassis_caster_z_offset" value="${2*0.0254}"/>
     <!-- Chassis Inertial Constants -->
-    <xacro:property name="chassis_mass" value="29.9371" />
-    <xacro:property name="com_x" value="${-4.0*0.0254}" />
-    <xacro:property name="com_y" value="0.0" />
-    <xacro:property name="com_z" value="${6.1875*0.0254-chassis_z_offset}" />
+    <xacro:property name="chassis_mass" value="29.9371"/>
+    <xacro:property name="com_x" value="${-4.0*0.0254}"/>
+    <xacro:property name="com_y" value="0.0"/>
+    <xacro:property name="com_z" value="${6.1875*0.0254-chassis_z_offset}"/>
 	<!-- Caster Constants -->
-    <xacro:property name="caster_x_offset" value="${-24.625*0.0254}" />
-    <xacro:property name="caster_radius" value="${3.5*0.0254}" />
-    <xacro:property name="caster_mass" value="0.1" />
+    <xacro:property name="caster_x_offset" value="${-24.625*0.0254}"/>
+    <xacro:property name="caster_radius" value="${3.5*0.0254}"/>
+    <xacro:property name="caster_mass" value="0.1"/>
 	<!-- Wheel Constants -->
-    <xacro:property name="wheel_radius" value="${6.1875*0.0254}" />
-    <xacro:property name="wheel_width" value="${4*0.0254}" />
-    <xacro:property name="wheel_mass" value="5" />
-    <xacro:property name="track_width" value="${31*0.0254}" />
+    <xacro:property name="wheel_radius" value="${6.1875*0.0254}"/>
+    <xacro:property name="wheel_width" value="${4*0.0254}"/>
+    <xacro:property name="wheel_mass" value="5"/>
+    <xacro:property name="track_width" value="${31*0.0254}"/>
     <!-- Lidar Constants -->
     <xacro:property name="lidar_height" value="${32.55*0.0254}"/>
@@ -39,8 +39,3 @@
     <xacro:property name="camera_x_offset" value="${(4+2.66916)*0.0254}"/>
     <xacro:property name="camera_z_offset" value="${(31-1.80395)*0.0254}"/>
-    <!-- IMU Constants -->
-    <xacro:property name="imu_mass" value="0.025"/>
-    <xacro:property name="imu_length" value="0.05"/>
-    <xacro:property name="imu_width" value="0.03"/>
-    <xacro:property name="imu_height" value="0.01"/>
 </robot>

File: marvin_simulation/urdf/marvin.xacro (robot description, xacro)
@@ -39,5 +39,5 @@
 	<!-- IMU -->
     <xacro:include filename="$(find common_xacro)/urdf/sensor/imu.xacro" />
-    <xacro:imu name="imu" mass="${imu_mass}" length="${imu_length}" width="${imu_width}" height="${imu_height}">
+    <xacro:imu name="imu">
 		<origin xyz="${-chassis_tower_length / 2 - chassis_electrical_length/2} 0 ${chassis_electrical_height}" rpy="0 0 0" />
     </xacro:imu>
