Commit message: Make Depth Camera dimension specific

File: common_xacro/urdf/sensor/depth_camera.xacro (robot description, xacro)
@@ -6,14 +6,15 @@
 <!-- Plugin: libgazebo_ros_camera.so (depth camera) -->
 <!-- Param name: the name of the depth camera. All published topics will start with /{name} -->
-<!-- Param mass: mass of the depth camera -->
-<!-- Param length: length of the depth camera -->
-<!-- Param width: width of the depth camera -->
-<!-- Param height: height of the depth camera -->
 <!-- Param parent: name of the parent link, defaulted to base_link -->
 <!-- Param joint_origin: location of the depth camera relative to parent link -->
 <robot xmlns:xacro="http://ros.org/wiki/xacro" name="depth_camera">
-    <xacro:macro name="depth_camera" params="name mass length width height parent:=base_link *joint_origin">
+    <xacro:macro name="depth_camera" params="name parent:=base_link *joint_origin">
         <!-- Includes -->
         <xacro:include filename="$(find common_xacro)/urdf/physics/inertia.xacro"/>
+        <!-- Constants -->
+        <xacro:property name="mass" value="0.230"/>
+        <xacro:property name="length" value="0.04310"/>
+        <xacro:property name="width" value="0.17525"/>
+        <xacro:property name="height" value="0.03025"/>
         <!-- Depth camera base link -->
         <link name="${name}_base_link" />

File: marvin_simulation/urdf/constants.xacro (robot description, xacro)
@@ -32,8 +32,4 @@
     <xacro:property name="lidar_height" value="${32.55*0.0254}"/>
     <!-- Camera Constants -->
-    <xacro:property name="camera_mass" value="0.230"/>
-    <xacro:property name="camera_length" value="0.04310"/>
-    <xacro:property name="camera_width" value="0.17525"/>
-    <xacro:property name="camera_height" value="0.03025"/>
     <xacro:property name="camera_angle" value="${10 * 0.01745327777}"/>
     <xacro:property name="camera_x_offset" value="${(4+2.66916)*0.0254}"/>

File: marvin_simulation/urdf/marvin.xacro (robot description, xacro)
@@ -29,5 +29,5 @@
     <!-- Camera -->
 	<xacro:include filename="$(find common_xacro)/urdf/sensor/depth_camera.xacro" />
-	<xacro:depth_camera name="zed" mass="${camera_mass}" length = "${camera_length}" width="${camera_width}" height="${camera_height}" parent="base_link">
+	<xacro:depth_camera name="zed">
 		<origin xyz="${camera_x_offset} 0 ${camera_z_offset}" rpy="0 ${camera_angle} 0" />
 	</xacro:depth_camera>
