Commit message: Make Caster dimension specific

File: common_xacro/urdf/wheel/caster.xacro (robot description, xacro)
@@ -5,12 +5,13 @@
 <!-- Joint Type: fixed -->
 <!-- Param name: the name of the caster -->
-<!-- Param mass: mass of the caster -->
-<!-- Param radius: radius of the caster -->
 <!-- Param parent: name of the parent link, defaulted to base_link -->
 <!-- Param joint_origin: location of the caster relative to parent link -->
 <robot xmlns:xacro="http://ros.org/wiki/xacro" name="caster">
-    <xacro:macro name="caster" params="name mass radius parent:=base_link *joint_origin">
+    <xacro:macro name="caster" params="name parent:=base_link *joint_origin">
         <!-- Includes -->
         <xacro:include filename="$(find common_xacro)/urdf/physics/inertia.xacro"/>
+        <!-- Constants -->
+        <xacro:property name="radius" value="${3.5*0.0254}"/>
+        <xacro:property name="mass" value="0.1"/>
         <!-- Caster link -->
         <link name="${name}_link">

File: marvin_simulation/urdf/constants.xacro (robot description, xacro)
@@ -22,11 +22,10 @@
 	<!-- Caster Constants -->
     <xacro:property name="caster_x_offset" value="${-24.625*0.0254}"/>
-    <xacro:property name="caster_radius" value="${3.5*0.0254}"/>
-    <xacro:property name="caster_mass" value="0.1"/>
+    <xacro:property name="caster_z_offset" value="${-0.875*0.0254}"/>
 	<!-- Wheel Constants -->
+    <xacro:property name="track_width" value="${31*0.0254}"/>
     <xacro:property name="wheel_radius" value="${6.1875*0.0254}"/>
     <xacro:property name="wheel_width" value="${4*0.0254}"/>
     <xacro:property name="wheel_mass" value="5"/>
-    <xacro:property name="track_width" value="${31*0.0254}"/>
     <!-- Lidar Constants -->
     <xacro:property name="lidar_height" value="${32.55*0.0254}"/>

File: marvin_simulation/urdf/marvin.xacro (robot description, xacro)
@@ -16,6 +16,6 @@
     <!-- Caster -->
     <xacro:include filename="$(find common_xacro)/urdf/wheel/caster.xacro"/>
-	<xacro:caster name="caster" mass="${caster_mass}" radius="${caster_radius}">
-        <origin xyz="${caster_x_offset} 0 ${caster_radius-chassis_z_offset}" rpy="0 0 0" />
+	<xacro:caster name="caster">
+        <origin xyz="${caster_x_offset} 0 ${caster_z_offset}" rpy="0 0 0" />
 	</xacro:caster>
     <!-- Wheels -->
