Commit message: Make Wheel dimension specific

File: common_xacro/urdf/wheel/wheel.xacro (robot description, xacro)
@@ -5,13 +5,14 @@
 <!-- Joint Type: continuous -->
 <!-- Param name: the name of the wheel -->
-<!-- Param mass: mass of the wheel -->
-<!-- Param radius: radius of the wheel -->
-<!-- Param width: width of the wheel -->
 <!-- Param parent: name of the parent link, defaulted to base_link -->
 <!-- Param joint_origin: location of the wheel relative to parent link -->
 <robot xmlns:xacro="http://ros.org/wiki/xacro" name="wheel">
-    <xacro:macro name="wheel" params="name mass radius width parent:=base_link *joint_origin">
+    <xacro:macro name="wheel" params="name parent:=base_link *joint_origin">
         <!-- Includes -->
         <xacro:include filename="$(find common_xacro)/urdf/physics/inertia.xacro"/>
+        <!-- Constants -->
+        <xacro:property name="radius" value="${6.1875*0.0254}"/>
+        <xacro:property name="width" value="${4*0.0254}"/>
+        <xacro:property name="mass" value="5"/>
         <!-- Wheel link -->
         <link name="${name}_link">

File: marvin_simulation/urdf/constants.xacro (robot description, xacro)
@@ -24,8 +24,6 @@
     <xacro:property name="caster_z_offset" value="${-0.875*0.0254}"/>
 	<!-- Wheel Constants -->
-    <xacro:property name="track_width" value="${31*0.0254}"/>
-    <xacro:property name="wheel_radius" value="${6.1875*0.0254}"/>
-    <xacro:property name="wheel_width" value="${4*0.0254}"/>
-    <xacro:property name="wheel_mass" value="5"/>
+    <xacro:property name="wheel_x_offset" value="${15.5*0.0254}"/>
+    <xacro:property name="wheel_z_offset" value="${1.8125*0.0254}"/>
     <!-- Lidar Constants -->
     <xacro:property name="lidar_height" value="${32.55*0.0254}"/>

File: marvin_simulation/urdf/marvin.xacro (robot description, xacro)
@@ -21,9 +21,9 @@
     <!-- Wheels -->
     <xacro:include filename="$(find common_xacro)/urdf/wheel/wheel.xacro"/>
-	<xacro:wheel name="right_wheel" mass="${wheel_mass}" radius="${wheel_radius}" width="${wheel_width}">
-		<origin xyz="0 -${track_width / 2} ${wheel_radius-chassis_z_offset}" rpy="0 0 0" />
+	<xacro:wheel name="right_wheel">
+		<origin xyz="0 ${-wheel_x_offset} ${wheel_z_offset}" rpy="0 0 0" />
 	</xacro:wheel>
-	<xacro:wheel name="left_wheel" mass="${wheel_mass}" radius="${wheel_radius}" width="${wheel_width}">
-		<origin xyz="0 ${track_width/2} ${wheel_radius-chassis_z_offset}" rpy="0 0 0" />
+	<xacro:wheel name="left_wheel">
+		<origin xyz="0 ${wheel_x_offset} ${wheel_z_offset}" rpy="0 0 0" />
 	</xacro:wheel>
     <!-- Camera -->
@@ -45,5 +45,5 @@
     <link name="encoder" />
 	<joint name="encoder_joint" type="fixed">
-		<origin xyz="0 0 ${wheel_radius-chassis_z_offset}" rpy="0 0 0" />
+		<origin xyz="0 0 ${wheel_z_offset}" rpy="0 0 0" />
 		<parent link="base_link" />
 		<child link="encoder" />

File: marvin_simulation/urdf/plugins.xacro (robot description, xacro)
@@ -8,6 +8,6 @@
 			<left_joint>left_wheel_joint</left_joint>
 			<right_joint>right_wheel_joint</right_joint>
-			<wheel_separation>${track_width}</wheel_separation>
-			<wheel_diameter>${2 * wheel_radius}</wheel_diameter>
+			<wheel_separation>${2 * wheel_x_offset}</wheel_separation>
+			<wheel_diameter>${2 * 6.1875*0.0254}</wheel_diameter>
 			<publish_tf>true</publish_tf>
 			<publish_wheel_tf>true</publish_wheel_tf>
